File: Microcontroller.kicad_sch (KiCad schematic)
At the start: 15 parts, among them SW3 SW_Push, U2 ESP32-C3-WROOM-02

Commit message: Routing improvement
Connections:
- net FREQ: now also U2.14 (IO19); no longer U2.18 (IO0)
- net IO0: now reaches R32.1
- net IO0: now also U2.18 (IO0); no longer U2.14 (IO19)
Changed lines of the file:
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@@
+	(wire
+		(pts
+			(xy 110.49 60.96) (xy 121.92 60.96)
+		)
+		(stroke
+			(width 0)
+			(type default)
+		)
+	)
 	(wire
 		(pts
@@
 	(wire
 		(pts
-			(xy 138.43 91.44) (xy 110.49 91.44)
-		)
-		(stroke
-			(width 0)
-			(type default)
-		)
-	)
-	(wire
-		(pts
 			(xy 149.86 83.82) (xy 146.05 83.82)
 		)
@@
 	(wire
 		(pts
+			(xy 110.49 91.44) (xy 121.92 91.44)
+		)
+		(stroke
+			(width 0)
+			(type default)
+		)
+	)
+	(wire
+		(pts
 			(xy 199.39 73.66) (xy 204.47 73.66)
 		)
@@
 	(wire
 		(pts
-			(xy 110.49 60.96) (xy 121.92 60.96)
+			(xy 133.35 91.44) (xy 138.43 91.44)
 		)
 		(stroke
@@
 	(label "EN"
 		(at 124.46 55.88 180)
+		(effects
+			(font
+				(size 1.27 1.27)
+			)
+			(justify right bottom)
+		)
+	)
+	(label "IO0"
+		(at 133.35 91.44 0)
+		(effects
+			(font
+				(size 1.27 1.27)
+			)
+			(justify left bottom)
+		)
+	)
+	(label "IO0"
+		(at 121.92 60.96 180)
 		(effects
 			(font
@@
 		)
 	)
-	(global_label "FREQ"
-		(shape input)
-		(at 121.92 60.96 0)
-		(fields_autoplaced yes)
-		(effects
-			(font
-				(size 1.27 1.27)
-			)
-			(justify left)
-		)
-		(property "Intersheetrefs" "${INTERSHEET_REFS}"
-			(at 129.7433 60.96 0)
-			(hide yes)
-			(show_name no)
-			(do_not_autoplace no)
-			(effects
-				(font
-					(size 1.27 1.27)
-				)
-				(justify left)
-			)
-		)
-	)
 	(global_label "LED0"
 		(shape input)
@@
 			)
 		)
+	)
+	(global_label "FREQ"
+		(shape input)
+		(at 121.92 91.44 0)
+		(fields_autoplaced yes)
+		(effects
+			(font
+				(size 1.27 1.27)
+			)
+			(justify left)
+		)
+		(property "Intersheetrefs" "${INTERSHEET_REFS}"
+			(at 129.7433 91.44 0)
+			(hide yes)
+			(show_name no)
+			(do_not_autoplace no)
+			(effects
+				(font
+					(size 1.27 1.27)
+				)
+				(justify left)
+			)
+		)
