File: iot-measurement-endpoint.kicad_pcb (KiCad board)
At the start: 4 copper layers, 55.3 x 39.5 mm, 98 parts, among them K1 Con_01x02, M1 Motor_DC, P1 USB_C_Plug_USB2.0, Q2 DMC2053UVT, Q3 DMC2053UVT, SW1 KMR232NG ULC LFS, SW2 KMR232NG ULC LFS, SW3 SW_Push, U1 CH330N, U2 ESP32-C3-WROOM-02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

Commit message: Adding resistance and capacitance connecting GND and Earth in the peripheral device
Parts:
- added C21: 47nF, Capacitor_SMD:C_0402_1005Metric, F.Cu at (114.9, 134.8)
- added R38: 1M, Resistor_SMD:R_0402_1005Metric, F.Cu at (116.9, 134.9)
Routing:
- net Earth: track 0.00 -> 4.24 mm
- net GND: vias 58 -> 60
